File: projects/moog-ladder-filter/moog-ladder-filter.kicad_sch (KiCad schematic)
At the start: 40 parts, among them J1 02x05_Eurorack_power, J2 IN1, J3 IN2, J4 CV_IN_FREQ, J5 IN2, Q1 MMDT3904, U1 SSI2144, U2 TL072

Commit message: update routing using AI
Parts:
- C10, C7, C8: footprint Eurorack:CAPPRD350W60D825H1300 -> Capacitor_SMD:C_0805_2012Metric
Other:
- moved on the sheet: D3
Changed lines of the file:
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@@
 	(wire
 		(pts
-			(xy 124.46 36.83) (xy 115.57 36.83)
+			(xy 124.46 36.83) (xy 113.03 36.83)
 		)
 		(stroke
@@
 	(wire
 		(pts
-			(xy 115.57 36.83) (xy 115.57 39.37)
+			(xy 113.03 36.83) (xy 113.03 39.37)
 		)
 		(stroke
@@
 	(wire
 		(pts
-			(xy 115.57 46.99) (xy 115.57 50.8)
+			(xy 113.03 46.99) (xy 113.03 50.8)
 		)
 		(stroke
@@
 			)
 		)
-		(property "Footprint" "Eurorack:CAPPRD350W60D825H1300"
+		(property "Footprint" "Capacitor_SMD:C_0805_2012Metric"
 			(at 205.74 127.3048 0)
 			(effects
@@
 	(symbol
 		(lib_id "Diode:1N4148WT")
-		(at 115.57 43.18 270)
+		(at 113.03 43.18 270)
 		(unit 1)
 		(exclude_from_sim no)
@@
 		(fields_autoplaced yes)
 		(property "Reference" "D3"
-			(at 118.11 41.9099 90)
+			(at 115.57 41.9099 90)
 			(effects
 				(font
@@
 		)
 		(property "Value" "1N4148WT"
-			(at 118.11 44.4499 90)
+			(at 115.57 44.4499 90)
 			(effects
 				(font
@@
 		)
 		(property "Footprint" "Diode_SMD:D_SOD-523"
-			(at 111.125 43.18 0)
+			(at 108.585 43.18 0)
 			(effects
 				(font
@@
 		)
 		(property "Datasheet" "https://www.diodes.com/assets/Datasheets/ds30396.pdf"
-			(at 115.57 43.18 0)
+			(at 113.03 43.18 0)
 			(effects
 				(font
@@
 		)
 		(property "Description" "75V 0.15A Fast switching Diode, SOD-523"
-			(at 115.57 43.18 0)
+			(at 113.03 43.18 0)
 			(effects
 				(font
@@
 		)
 		(property "Sim.Device" "D"
-			(at 115.57 43.18 0)
+			(at 113.03 43.18 0)
 			(effects
 				(font
@@
 		)
 		(property "Sim.Pins" "1=K 2=A"
-			(at 115.57 43.18 0)
+			(at 113.03 43.18 0)
 			(effects
 				(font
@@
 	(symbol
 		(lib_id "power:GND")
-		(at 115.57 50.8 0)
+		(at 113.03 50.8 0)
 		(unit 1)
 		(exclude_from_sim no)
@@
 		(fields_autoplaced yes)
 		(property "Reference" "#PWR08"
-			(at 115.57 57.15 0)
+			(at 113.03 57.15 0)
 			(effects
 				(font
@@
 		)
 		(property "Value" "GND"
-			(at 115.57 55.88 0)
+			(at 113.03 55.88 0)
 			(effects
 				(font
@@
 		)
 		(property "Footprint" ""
-			(at 115.57 50.8 0)
+			(at 113.03 50.8 0)
 			(effects
 				(font
@@
 		)
 		(property "Datasheet" ""
-			(at 115.57 50.8 0)
+			(at 113.03 50.8 0)
 			(effects
 				(font
@@
 		)
 		(property "Description" "Power symbol creates a global label with name \"GND\" , ground"
-			(at 115.57 50.8 0)
+			(at 113.03 50.8 0)
 			(effects
 				(font
@@
 			)
 		)
-		(property "Footprint" "Eurorack:CAPPRD350W60D825H1300"
+		(property "Footprint" "Capacitor_SMD:C_0805_2012Metric"
 			(at 52.07 48.5648 0)
 			(effects
@@
 			)
 		)
-		(property "Footprint" "Eurorack:CAPPRD350W60D825H1300"
+		(property "Footprint" "Capacitor_SMD:C_0805_2012Metric"
 			(at 52.07 25.7048 0)
 			(effects
@@
 			(effects
 				(font
+					(size 1.27 1.27)
+				)
+				(hide yes)
+			)
+		)
+		(property "MPN" ""
+			(at 48.26 26.67 90)
+			(effects
+				(font
